File: _saved_pd_tia.sch (KiCad schematic (older format))
At the start: 21 parts, among them P1 BNC, U1 ED2610, U2 LM2940, U3 OPA2211

Commit message: Autorouter found a solution, but on a bigger board
Parts:
- P1: footprint (none) -> footprints:Dual-BNC-ARF2136
- U3: footprint (none) -> Housings_SOIC:SOIC-8-1EP_3.9x4.9mm_Pitch1.27mm
Changed lines of the file:
@@
 $EndComp
 $Comp
-L PWR_FLAG #FLG2
+L PWR_FLAG #FLG01
 U 1 1 58C03418
 P 2350 1200
-F 0 "#FLG2" H 2350 1295 50  0001 C CNN
+F 0 "#FLG01" H 2350 1295 50  0001 C CNN
 F 1 "PWR_FLAG" H 2350 1380 50  0000 C CNN
 F 2 "" H 2350 1200 50  0000 C CNN
@@
 $EndComp
 $Comp
-L PWR_FLAG #FLG3
+L PWR_FLAG #FLG02
 U 1 1 58C0343C
 P 2350 2000
-F 0 "#FLG3" H 2350 2095 50  0001 C CNN
+F 0 "#FLG02" H 2350 2095 50  0001 C CNN
 F 1 "PWR_FLAG" H 2350 2180 50  0000 C CNN
 F 2 "" H 2350 2000 50  0000 C CNN
@@
 $EndComp
 $Comp
-L PWR_FLAG #FLG1
+L PWR_FLAG #FLG03
 U 1 1 58C036F3
 P 1950 2000
-F 0 "#FLG1" H 1950 2095 50  0001 C CNN
+F 0 "#FLG03" H 1950 2095 50  0001 C CNN
 F 1 "PWR_FLAG" H 1950 2180 50  0000 C CNN
 F 2 "" H 1950 2000 50  0000 C CNN
@@
 $EndComp
 $Comp
-L +15V #PWR8
+L +15V #PWR04
 U 1 1 58C0379C
 P 2750 1200
-F 0 "#PWR8" H 2750 1050 50  0001 C CNN
+F 0 "#PWR04" H 2750 1050 50  0001 C CNN
 F 1 "+15V" H 2750 1340 50  0000 C CNN
 F 2 "" H 2750 1200 50  0000 C CNN
@@
 $EndComp
 $Comp
-L GND #PWR2
+L GND #PWR05
 U 1 1 58C03A65
 P 2000 1650
-F 0 "#PWR2" H 2000 1400 50  0001 C CNN
+F 0 "#PWR05" H 2000 1400 50  0001 C CNN
 F 1 "GND" H 2000 1500 50  0000 C CNN
 F 2 "" H 2000 1650 50  0000 C CNN
@@
 $EndComp
 $Comp
-L +15V #PWR11
+L +15V #PWR06
 U 1 1 58C03C50
 P 3350 1600
-F 0 "#PWR11" H 3350 1450 50  0001 C CNN
+F 0 "#PWR06" H 3350 1450 50  0001 C CNN
 F 1 "+15V" H 3350 1740 50  0000 C CNN
 F 2 "" H 3350 1600 50  0000 C CNN
@@
 $EndComp
 $Comp
-L GND #PWR12
+L GND #PWR07
 U 1 1 58C04081
 P 3350 2100
-F 0 "#PWR12" H 3350 1850 50  0001 C CNN
+F 0 "#PWR07" H 3350 1850 50  0001 C CNN
 F 1 "GND" H 3350 1950 50  0000 C CNN
 F 2 "" H 3350 2100 50  0000 C CNN
@@
 $EndComp
 $Comp
-L GND #PWR14
+L GND #PWR08
 U 1 1 58C04900
 P 4350 1200
-F 0 "#PWR14" H 4350 950 50  0001 C CNN
+F 0 "#PWR08" H 4350 950 50  0001 C CNN
 F 1 "GND" H 4350 1050 50  0000 C CNN
 F 2 "" H 4350 1200 50  0000 C CNN
@@
 $EndComp
 $Comp
-L +9V #PWR15
+L +9V #PWR09
 U 1 1 58C05942
 P 4950 1600
-F 0 "#PWR15" H 4950 1450 50  0001 C CNN
+F 0 "#PWR09" H 4950 1450 50  0001 C CNN
 F 1 "+9V" H 4950 1740 50  0000 C CNN
 F 2 "" H 4950 1600 50  0000 C CNN
@@
 $EndComp
 $Comp
-L +9V #PWR4
+L +9V #PWR010
 U 1 1 58C05CB8
 P 2150 3900
-F 0 "#PWR4" H 2150 3750 50  0001 C CNN
+F 0 "#PWR010" H 2150 3750 50  0001 C CNN
 F 1 "+9V" H 2150 4040 50  0000 C CNN
 F 2 "" H 2150 3900 50  0000 C CNN
@@
 	2000 3550 2000 3600
 $Comp
-L GND #PWR1
+L GND #PWR011
 U 1 1 58C06181
 P 1300 3550
-F 0 "#PWR1" H 1300 3300 50  0001 C CNN
+F 0 "#PWR011" H 1300 3300 50  0001 C CNN
 F 1 "GND" H 1300 3400 50  0000 C CNN
 F 2 "" H 1300 3550 50  0000 C CNN
@@
 F 0 "U3" H 3850 3300 50  0000 L CNN
 F 1 "OPA2211" H 3850 3000 50  0000 L CNN
-F 2 "" H 3750 3200 50  0000 C CNN
+F 2 "Housings_SOIC:SOIC-8-1EP_3.9x4.9mm_Pitch1.27mm" H 3750 3200 50  0001 C CNN
 F 3 "" H 3850 3300 50  0000 C CNN
 	2    3850 3150
@@
 	2150 3450 2400 3450
 $Comp
-L GND #PWR3
+L GND #PWR012
 U 1 1 58C06E7E
 P 2150 3250
-F 0 "#PWR3" H 2150 3000 50  0001 C CNN
+F 0 "#PWR012" H 2150 3000 50  0001 C CNN
 F 1 "GND" H 2150 3100 50  0000 C CNN
 F 2 "" H 2150 3250 50  0000 C CNN
@@
 $EndComp
 $Comp
-L GND #PWR10
+L GND #PWR013
 U 1 1 58C07E0C
 P 3100 2950
-F 0 "#PWR10" H 3100 2700 50  0001 C CNN
+F 0 "#PWR013" H 3100 2700 50  0001 C CNN
 F 1 "GND" H 3100 2800 50  0000 C CNN
 F 2 "" H 3100 2950 50  0000 C CNN
@@
 	2950 2950 3100 2950
 $Comp
-L +15V #PWR5
+L +15V #PWR014
 U 1 1 58C07FF7
 P 2600 2850
-F 0 "#PWR5" H 2600 2700 50  0001 C CNN
+F 0 "#PWR014" H 2600 2700 50  0001 C CNN
 F 1 "+15V" H 2600 2990 50  0000 C CNN
 F 2 "" H 2600 2850 50  0000 C CNN
@@
 Connection ~ 2600 3700
 $Comp
-L GND #PWR9
+L GND #PWR015
 U 1 1 58C08E6F
 P 2950 3750
-F 0 "#PWR9" H 2950 3500 50  0001 C CNN
+F 0 "#PWR015" H 2950 3500 50  0001 C CNN
 F 1 "GND" H 2950 3600 50  0000 C CNN
 F 2 "" H 2950 3750 50  0000 C CNN
@@
 	2950 3700 2950 3750
 $Comp
-L GND #PWR13
+L GND #PWR016
 U 1 1 58C093FA
 P 3400 3050
-F 0 "#PWR13" H 3400 2800 50  0001 C CNN
+F 0 "#PWR016" H 3400 2800 50  0001 C CNN
 F 1 "GND" H 3400 2900 50  0000 C CNN
 F 2 "" H 3400 3050 50  0000 C CNN
@@
 F 0 "P1" H 5160 3270 50  0000 C CNN
 F 1 "BNC" V 5260 3090 50  0000 C CNN
-F 2 "" H 5150 3150 50  0000 C CNN
+F 2 "footprints:Dual-BNC-ARF2136" H 5150 3150 50  0001 C CNN
 F 3 "" H 5150 3150 50  0000 C CNN
 	1    5150 3150
@@
 	4900 3150 5000 3150
 $Comp
-L GND #PWR16
+L GND #PWR017
 U 1 1 58C0A587
 P 5150 3400
-F 0 "#PWR16" H 5150 3150 50  0001 C CNN
+F 0 "#PWR017" H 5150 3150 50  0001 C CNN
 F 1 "GND" H 5150 3250 50  0000 C CNN
 F 2 "" H 5150 3400 50  0000 C CNN
